File: Block Diagram.kicad_sch (KiCad schematic)
At the start: 0 parts

Commit message: Frist draft of Schematic
Other:
- note added: "3v3"
- note added: "5V"
- note added: "Buttons for control [1xN]"
- note added: "LED Array [1XN]"
- note added: "MCU"
- note removed: "+??V"
- note removed: "+A3V3"
