File: pomodoroTimer_v2.kicad_sch (KiCad schematic)
At the start: 0 parts

Commit message: update f
Other:
- removed sheet Power - Sequencing
Changed lines of the file:
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@@
-	)
-	(sheet
-		(at 340.36 313.69)
-		(size 35.56 5.08)
-		(exclude_from_sim no)
-		(in_bom yes)
-		(on_board yes)
-		(dnp no)
-		(stroke
-			(width 0.1524)
-			(type solid)
-		)
-		(fill
-			(color 0 0 0 0.0000)
-		)
-		(property "Sheetname" "Power - Sequencing"
-			(at 340.36 312.6609 0)
-			(effects
-				(font
-					(face "Times New Roman")
-					(size 1.905 1.905)
-					(bold yes)
-					(color 0 0 0 1)
-				)
-				(justify left bottom)
-			)
-		)
-		(property "Sheetfile" "Power - Sequencing.kicad_sch"
-			(at 341.63 314.96 0)
-			(effects
-				(font
-					(face "Arial")
-					(size 1.27 1.27)
-				)
-				(justify left top)
-			)
-		)
-		(instances
-			(project "pomodoroTimer_v2"
-				(path "/f9e05184-c88b-4a88-ae9c-ab2bdb32be7c"
-					(page "7")
-				)
-			)
-		)
 	)
 	(sheet
